Commit message: fix repository

File: urdf/m2wr_arm2.xacro (robot description, xacro)
@@ -300,63 +300,3 @@
   	<child link="left_grip_link"/>
   </joint>
-<transmission name="arm_joint_01_trans">
-	<type>transmission_interface/SimpleTransmission</type>
-	<joint name="arm_joint_01">
-		<hardwareInterface>hardware_interface/EffortJointInterface</hardwareInterface>
-	</joint>
-	<actuator name="motor1">
-		<hardwareInterface>hardware_interface/EffortJointInterface</hardwareInterface>
-		<mechanicalInterface>1</mechanicalInterface>
-	</actuator>
-</transmission>
-<transmission name="arm_joint_02_trans">
-	<type>transmission_interface/SimpleTransmission</type>
-	<joint name="arm_joint_02">
-		<hardwareInterface>hardware_interface/EffortJointInterface</hardwareInterface>
-	</joint>
-	<actuator name="motor2">
-		<hardwareInterface>hardware_interface/EffortJointInterface</hardwareInterface>
-		<mechanicalInterface>1</mechanicalInterface>
-	</actuator>
-</transmission>
-<transmission name="arm_joint_03_trans">
-	<type>transmission_interface/SimpleTransmission</type>
-	<joint name="arm_joint_03">
-		<hardwareInterface>hardware_interface/EffortJointInterface</hardwareInterface>
-	</joint>
-	<actuator name="motor3">
-		<hardwareInterface>hardware_interface/EffortJointInterface</hardwareInterface>
-		<mechanicalInterface>1</mechanicalInterface>
-	</actuator>
-</transmission>
-<transmission name="arm_joint_04_trans">
-	<type>transmission_interface/SimpleTransmission</type>
-	<joint name="arm_joint_04">
-		<hardwareInterface>hardware_interface/EffortJointInterface</hardwareInterface>
-	</joint>
-	<actuator name="motor4">
-		<hardwareInterface>hardware_interface/EffortJointInterface</hardwareInterface>
-		<mechanicalInterface>1</mechanicalInterface>
-	</actuator>
-</transmission>
-<transmission name="left_grip_trans">
-	<type>transmission_interface/SimpleTransmission</type>
-	<joint name="left_grip_joint">
-		<hardwareInterface>hardware_interface/EffortJointInterface</hardwareInterface>
-	</joint>
-	<actuator name="motor5">
-		<hardwareInterface>hardware_interface/EffortJointInterface</hardwareInterface>
-		<mechanicalInterface>1</mechanicalInterface>
-	</actuator>
-</transmission>
-<transmission name="right_grip_trans">
-	<type>transmission_interface/SimpleTransmission</type>
-	<joint name="right_grip_joint">
-		<hardwareInterface>hardware_interface/EffortJointInterface</hardwareInterface>
-	</joint>
-	<actuator name="motor6">
-		<hardwareInterface>hardware_interface/EffortJointInterface</hardwareInterface>
-		<mechanicalInterface>1</mechanicalInterface>
-	</actuator>
-</transmission>
 </robot>

File: urdf/robot5.xacro (robot description, xacro)
@@ -87,16 +87,4 @@
     </visual>
   </link>
-  <link name="link_right_wheel_back">
-    <xacro:default_inertial mass="0.2"/>
-    <collision name="link_right_wheel_collision_back">
-      <origin rpy="0 1.5707 1.5707" xyz="0 0 0"/>
-      <xacro:wheel_geometry />
-    </collision>
-    <visual name="link_right_wheel_visual_back">
-      <origin rpy="0 1.5707 1.5707" xyz="0 0 0"/>
-      <xacro:wheel_geometry />
-      <material name="red"/>
-    </visual>
-  </link>
    <link name="link_left_wheel">
     <xacro:default_inertial mass="0.2"/>
@@ -111,18 +99,6 @@
     </visual>
   </link>
-     <link name="link_left_wheel_back">
-    <xacro:default_inertial mass="0.2"/>
-    <collision name="link_left_wheel_collision_back">
-      <origin rpy="0 1.5707 1.5707" xyz="0 0 0"/>
-      <xacro:wheel_geometry />
-    </collision>
-    <visual name="link_left_wheel_visual_back">
-      <origin rpy="0 1.5707 1.5707" xyz="0 0 0"/>
-      <xacro:wheel_geometry />
-      <material name="red"/>
-    </visual>
-  </link>
   <joint name="joint_right_wheel" type="continuous">
-    <origin rpy="0 0 0" xyz="0.2 0.15 0"/>
+    <origin rpy="0 0 0" xyz="-0.05 0.15 0"/>
     <child link="link_right_wheel"/>
     <parent link="link_chassis"/>
@@ -131,14 +107,6 @@
     <joint_properties damping="1.0" friction="1.0"/>
   </joint>
-    <joint name="joint_right_wheel_back" type="continuous">
-    <origin rpy="0 0 0" xyz="-0.2 0.15 0"/>
-    <child link="link_right_wheel_back"/>
-    <parent link="link_chassis"/>
-    <axis rpy="0 0 0" xyz="0 1 0"/>
-    <limit effort="10000" velocity="1000"/>
-    <joint_properties damping="1.0" friction="1.0"/>
-  </joint>
   <joint name="joint_left_wheel" type="continuous">
-    <origin rpy="0 0 0" xyz="0.2 -0.15 0"/>
+    <origin rpy="0 0 0" xyz="-0.05 -0.15 0"/>
     <child link="link_left_wheel"/>
     <parent link="link_chassis"/>
@@ -147,26 +115,11 @@
     <joint_properties damping="1.0" friction="1.0"/>
   </joint>
-  <joint name="joint_left_wheel_back" type="continuous">
-    <origin rpy="0 0 0" xyz="-0.2 -0.15 0"/>
-    <child link="link_left_wheel_back"/>
-    <parent link="link_chassis"/>
-    <axis rpy="0 0 0" xyz="0 1 0"/>
-    <limit effort="10000" velocity="1000"/>
-    <joint_properties damping="1.0" friction="1.0"/>
-  </joint>
-  <joint name="hokuyo_joint" type="fixed">
-    <axis xyz="0 1 0" />
-    <origin xyz="-0.05 -0.15 0" rpy="0 0 0"/>
-    <parent link="link_chassis"/>
-    <child link="hokuyo_link"/>
-  </joint>
-  <!-- Hokuyo Laser -->
-  <link name="hokuyo_link">
-    <collision>
-      <origin xyz="0 0 0.025" rpy="0 0 0"/>
-      <geometry>
-    <box size="0.1 0.1 0.1"/>
-      </geometry>
-    </collision>
+  <link name="camera_link">
+	    <collision>
+	      <origin xyz="0 0 0.1" rpy="0 0 0"/>
+	      <geometry>
+		<box size="0.05 0.05 0.2"/>
+	      </geometry>
+	    </collision>
 	    <visual>
 	      <origin xyz="0 0 0.025" rpy="0 0 0"/>
@@ -178,9 +131,15 @@
 	      </material>
 	    </visual>
-    <inertial>
-      <mass value="1e-5" />
-      <origin xyz="0 0 0" rpy="0 0 0"/>
-      <inertia ixx="1e-6" ixy="0" ixz="0" iyy="1e-6" iyz="0" izz="1e-6" />
-    </inertial>
+	    <inertial>
+	      <mass value="1e-5" />
+	      <origin xyz="0 0 0" rpy="0 0 0"/>
+	      <inertia ixx="1e-6" ixy="0" ixz="0" iyy="1e-6" iyz="0" izz="1e-6" />
+	    </inertial>
   </link>
+  <joint name="camera_joint" type="fixed">
+	    <axis xyz="0 1 0" />
+	    <origin xyz="0.23 0 0.235" rpy="0 0 0"/>
+	    <parent link="link_chassis"/>
+	    <child link="camera_link"/>
+	 </joint>
 </robot>
